File: hw/sch_pcb/PCRD06A.kicad_pcb (KiCad board)
At the start: 2 copper layers, 50.3 x 40.1 mm, 33 parts, among them J1 3.6V, J2 HEADER_2x01_PARALLEL, J3 HEADER_2x01_PARALLEL, J5 HEADER_2x01_PARALLEL, J6 HEADER_2x01_PARALLEL, J7 HEADER_2x01_PARALLEL, J8 HEADER_2x03_PARALLEL, M1 HOLE, M2 HOLE, M3 HOLE, M4 HOLE, M5 HOLE, U1 TS3021ILT, U2 AD8691, U5 TS5A4594

Commit message: Přegenerování výrobních dat.
Other:
- net class Default removed
- net class MLAB_default removed
- net class MLAB_power removed
