File: hw/sch_pcb/PCRD06A.kicad_sch (KiCad schematic)
At the start: 33 parts, among them J1 3.6V, J2 HEADER_2x01_PARALLEL, J3 HEADER_2x01_PARALLEL, J5 HEADER_2x01_PARALLEL, J6 HEADER_2x01_PARALLEL, J7 HEADER_2x01_PARALLEL, J8 HEADER_2x03_PARALLEL, M1 HOLE, M2 HOLE, M3 HOLE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

Commit message: Update documentation.
Other:
- title: NAME -> PCRD06A
